File: pcb/rgb2vga.kicad_pcb (KiCad board)
At the start: 2 copper layers, 70.5 x 55.9 mm, 44 parts, among them J1 GPIO_0, J2 RGB_IN, J3 COCO3_RGB_IN, J4 C_VIDEO_IN, J5 GPIO_1, J6 VGA_OUT, J7 Conn_01x03_Male, SW1 SW_DIP_x10, SW2 SW_DP3T, U1 LM1881

Commit message: fiducials, pics
Parts:
- added JP1: lowpass, 000_LOCAL:JP_0805, F.Cu at (150.1, 93.9)
- added REF**: Fiducial_1mm_Mask2mm, 000_LOCAL:Fiducial_1mm_Mask2mm, F.Cu at (176.1, 75.6)
- added REF**: Fiducial_1mm_Mask2mm, 000_LOCAL:Fiducial_1mm_Mask2mm, F.Cu at (110.3, 126.6)
- added REF**: Fiducial_1mm_Mask2mm, 000_LOCAL:Fiducial_1mm_Mask2mm, F.Cu at (176.1, 126.6)
- R29: footprint 000_LOCAL:R_0805_SJC -> 000_LOCAL:R_0805
Other:
- board text added: "C_VIDEO 500khz lowpass"
- board text added: "cut"
- board text removed: "500khz lowpass"

Commit message: pics
Other:
- board text added: "500khz lowpass"
- board text removed: "C_VIDEO 500khz lowpass"

Commit message: C4 510p, dnp fiducials, pnp export
Parts:
- C4: value 512p -> 510p

Commit message: export bom, centroid
Parts:
- J1: value GPIO_0 -> PinSocket_02x20_P2.54mm_Vertical_tht
- J2: value RGB_IN -> HD15F_horizontal_tht
- J3: value COCO3_RGB_IN -> IDC-Header_2x05_P2.54mm_Horizontal_tht
- J4: value C_VIDEO_IN -> RCA_horizontal_tht
- J5: value GPIO_1 -> PinSocket_02x20_P2.54mm_Vertical_tht
- J6: value VGA_OUT -> HD15F_horizontal_tht
