File: pcb/rgb2vga.kicad_pcb (KiCad board)
At the start: 2 copper layers, 70.5 x 55.9 mm, 48 parts, among them J1 PinSocket_02x20_P2.54mm_Verti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, J2 HD15F_horizontal_tht, J3 IDC-Header_2x05_P2.54mm_Horiz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, J4 RCA_horizontal_tht, J5 PinSocket_02x20_P2.54mm_Verti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, J6 HD15F_horizontal_tht, J7 Conn_01x03_Male, SW1 SW_DIP_x10, SW2 SW_DP3T, U1 LM1881

Commit message: silkscreen & pics
Other:
- board text added: "ADC TRIM"
- board text removed: "DAC TRIM"
Changed lines of the file:
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@@
 	(title_block
 		(title "DE0-NANO_RGB2VGA")
-		(date "2024-08-06")
-		(rev "017")
+		(date "2024-08-30")
+		(rev "018")
 		(company "Brian K. White - b.kenyon.w@gmail.com")
 		(comment 1 "github.com/bkw777/rgb2vga")
@@
 		)
 	)
-	(gr_text "DAC TRIM"
+	(gr_text "ADC TRIM"
 		(at 156.2735 128.27 270)
 		(layer "B.SilkS")
@@
 		)
 	)
-	(gr_text "DAC\nTRIM"
+	(gr_text "ADC\nTRIM"
 		(at 152.3365 127.127 0)
 		(layer "F.SilkS")

Commit message: rename msx switch to offset
Connections:
- net /SW_MSX renamed /SW_OFFSET
Other:
- board text added: "OFFSET"
- board text removed: "MSX"
